File: board/board2.sch (KiCad schematic (older format))
At the start: 86 parts, among them J1 Battery, J2 Serial, J3 SWD, J4 Range_Front, J5 Range_Left, J6 Range_Right, J7 POWER, J8 EXP, SW1 RST, SW2 Left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

Commit message: Calc target angle, then PID on that angle instead of PID on the distance
Helps make sure it is facing the right direction when close to the path
Parts:
- J3: symbol Connector:Conn_ARM_JTAG_SWD_10 -> board2-rescue:Conn_ARM_JTAG_SWD_10-Connector
- U4, U5: symbol Motor:Motor_Encoder_Pololu -> board2-rescue:Motor_Encoder_Pololu-Motor
- U7: symbol Sensor_Motion:MPU-6500 -> board2-rescue:MPU-6500-Sensor_Motion
Changed lines of the file:
@@
 EESchema Schematic File Version 4
 LIBS:board2-cache
-EELAYER 29 0
+EELAYER 30 0
 EELAYER END
 $Descr USLetter 11000 8500
@@
 	3650 5650 4000 5650
 $Comp
-L Connector:Conn_ARM_JTAG_SWD_10 J3
+L board2-rescue:Conn_ARM_JTAG_SWD_10-Connector J3
 U 1 1 5C4439E0
 P 1050 5450
@@
 $EndComp
 $Comp
-L Sensor_Motion:MPU-6500 U7
+L board2-rescue:MPU-6500-Sensor_Motion U7
 U 1 1 5CF8B427
 P 8900 5750
@@
 	9750 1750 9750 1800
 $Comp
-L Motor:Motor_Encoder_Pololu U5
+L board2-rescue:Motor_Encoder_Pololu-Motor U5
 U 1 1 5C471455
 P 9750 3100
@@
 $EndComp
 $Comp
-L Motor:Motor_Encoder_Pololu U4
+L board2-rescue:Motor_Encoder_Pololu-Motor U4
 U 1 1 5C4713FB
 P 9750 2200
